Commit message: Update

File: packages/simdemo/config/robot.urdf.xacro (robot description, xacro)
@@ -83,4 +83,29 @@
     <mu2>0.01</mu2>
   </gazebo>
+  <link name="lidar_link">
+    <visual>
+      <geometry><cylinder radius="0.05" length="0.04"/></geometry>
+    </visual>
+    <inertial>
+      <mass value="0.1"/>
+      <inertia ixx="0.0001" ixy="0" ixz="0" iyy="0.0001" iyz="0" izz="0.0001"/>
+    </inertial>
+  </link>
+  <joint name="lidar_joint" type="fixed">
+    <parent link="base_link"/>
+    <child link="lidar_link"/>
+    <origin xyz="0.1 0 0.1"/>
+  </joint>
+  <link name="imu_link">
+    <inertial>
+      <mass value="0.01"/>
+      <inertia ixx="1e-5" ixy="0" ixz="0" iyy="1e-5" iyz="0" izz="1e-5"/>
+    </inertial>
+  </link>
+  <joint name="imu_joint" type="fixed">
+    <parent link="base_link"/>
+    <child link="imu_link"/>
+    <origin xyz="-0.1 0 0.05"/>
+  </joint>
   <ros2_control name="GazeboSimSystem" type="system">
     <hardware>
@@ -103,3 +128,46 @@
     </plugin>
   </gazebo>
+  <gazebo reference="lidar_link">
+    <sensor name="gpu_lidar" type="gpu_lidar">
+      <gz_frame_id>lidar_link</gz_frame_id>
+      <pose>0 0 0 0 0 0</pose>
+      <topic>scan</topic>
+      <update_rate>10</update_rate>
+      <lidar>
+        <scan>
+          <horizontal>
+            <samples>640</samples>
+            <resolution>1</resolution>
+            <min_angle>-3.14159</min_angle>
+            <max_angle>3.14159</max_angle>
+          </horizontal>
+        </scan>
+        <range>
+          <min>0.08</min>
+          <max>10.0</max>
+          <resolution>0.01</resolution>
+        </range>
+      </lidar>
+      <visualize>true</visualize>
+    </sensor>
+  </gazebo>
+  <gazebo reference="imu_link">
+    <sensor name="imu" type="imu">
+      <always_on>1</always_on>
+      <update_rate>50</update_rate>
+      <visualize>true</visualize>
+      <topic>imu</topic>
+      <enable_metrics>true</enable_metrics>
+      <gz_frame_id>imu_link</gz_frame_id>
+    </sensor>
+  </gazebo>
+  <gazebo>
+    <plugin
+      filename="gz-sim-odometry-publisher-system"
+      name="gz::sim::systems::OdometryPublisher">
+      <dimensions>3</dimensions>
+      <odom_topic>/sim/odom</odom_topic>
+      <tf_topic>/sim/odom/tf</tf_topic>
+    </plugin>
+  </gazebo>
 </robot>

Commit message: Update

File: packages/simdemo/config/robot.urdf.xacro (robot description, xacro)
@@ -95,5 +95,5 @@
     <parent link="base_link"/>
     <child link="lidar_link"/>
-    <origin xyz="0.1 0 0.1"/>
+    <origin xyz="0.1 0 0.15"/>
   </joint>
   <link name="imu_link">
@@ -148,6 +148,11 @@
           <resolution>0.01</resolution>
         </range>
+        <noise>
+          <type>gaussian</type>
+          <mean>0.0</mean>
+          <stddev>0.01</stddev>
+        </noise>
       </lidar>
-      <visualize>true</visualize>
+      <visualize>false</visualize>
     </sensor>
   </gazebo>
@@ -156,5 +161,5 @@
       <always_on>1</always_on>
       <update_rate>50</update_rate>
-      <visualize>true</visualize>
+      <visualize>false</visualize>
       <topic>imu</topic>
       <enable_metrics>true</enable_metrics>
